File: KiCAD/Wecker.sch (KiCad schematic (older format))
At the start: 4 parts

Commit message: Platinenlayout ausprobiert
Parts:
- 33µ1: renamed from 33µ; footprint (none) -> Capacitors_ThroughHole:C_Radial_D5_L6_P2.5
- 47µ1: renamed from 47µ; footprint (none) -> Capacitors_ThroughHole:C_Axial_D6_L11_P18
- Atmega328P1: renamed from IC?; footprint DIL28 -> Pin_Headers:Pin_Header_Straight_2x14
- U1: renamed from U?; footprint (none) -> Connect:PINHEAD1-3
Connections:
- net +3V3 is gone; now on net VCC: Atmega328P1.20 (AVCC), Atmega328P1.21 (AREF), Atmega328P1.7 (VCC)
Changed lines of the file:
@@
 LIBS:contrib
 LIBS:valves
+LIBS:Wecker-cache
 EELAYER 25 0
 EELAYER END
@@
 $EndDescr
 $Comp
-L ATMEGA328P-P IC?
+L ATMEGA328P-P Atmega328P1
 U 1 1 5627CFEE
 P 5750 3150
-F 0 "IC?" H 5000 4400 40  0000 L BNN
+F 0 "Atmega328P1" H 5000 4400 40  0000 L BNN
 F 1 "ATMEGA328P-P" H 6150 1750 40  0000 L BNN
-F 2 "DIL28" H 5750 3150 30  0000 C CIN
+F 2 "Pin_Headers:Pin_Header_Straight_2x14" H 5750 3150 30  0000 C CIN
 F 3 "" H 5750 3150 60  0000 C CNN
 	1    5750 3150
@@
 $EndComp
 $Comp
-L GND #PWR?
+L GND #PWR01
 U 1 1 5627D0F9
 P 4250 4350
-F 0 "#PWR?" H 4250 4100 50  0001 C CNN
+F 0 "#PWR01" H 4250 4100 50  0001 C CNN
 F 1 "GND" H 4250 4200 50  0000 C CNN
 F 2 "" H 4250 4350 60  0000 C CNN
@@
 $EndComp
 $Comp
-L +3.3V #PWR?
+L VCC #PWR02
 U 1 1 5627D148
 P 4250 2000
-F 0 "#PWR?" H 4250 1850 50  0001 C CNN
-F 1 "+3.3V" H 4250 2140 50  0000 C CNN
+F 0 "#PWR02" H 4250 1850 50  0001 C CNN
+F 1 "VCC" H 4250 2140 50  0000 C CNN
 F 2 "" H 4250 2000 60  0000 C CNN
 F 3 "" H 4250 2000 60  0000 C CNN
@@
 Connection ~ 4250 2350
 $Comp
-L +5V #PWR?
+L +5V #PWR03
 U 1 1 5627D248
 P 1400 1100
-F 0 "#PWR?" H 1400 950 50  0001 C CNN
+F 0 "#PWR03" H 1400 950 50  0001 C CNN
 F 1 "+5V" H 1400 1240 50  0000 C CNN
 F 2 "" H 1400 1100 60  0000 C CNN
@@
 $EndComp
 $Comp
-L 7805 U?
+L 7805 U1
 U 1 1 5627D26A
 P 2050 1150
-F 0 "U?" H 2200 954 60  0000 C CNN
+F 0 "U1" H 2200 954 60  0000 C CNN
 F 1 "7805" H 2050 1350 60  0000 C CNN
-F 2 "" H 2050 1150 60  0000 C CNN
+F 2 "Connect:PINHEAD1-3" H 2050 1150 60  0001 C CNN
 F 3 "" H 2050 1150 60  0000 C CNN
 	1    2050 1150
@@
 	1400 1100 1650 1100
 $Comp
-L VCC #PWR?
+L VCC #PWR04
 U 1 1 5627D2D0
 P 2450 1100
-F 0 "#PWR?" H 2450 950 50  0001 C CNN
+F 0 "#PWR04" H 2450 950 50  0001 C CNN
 F 1 "VCC" H 2450 1250 50  0000 C CNN
 F 2 "" H 2450 1100 60  0000 C CNN
@@
 $EndComp
 $Comp
-L GND #PWR?
+L GND #PWR05
 U 1 1 5627D2E8
 P 2050 1550
-F 0 "#PWR?" H 2050 1300 50  0001 C CNN
+F 0 "#PWR05" H 2050 1300 50  0001 C CNN
 F 1 "GND" H 2050 1400 50  0000 C CNN
 F 2 "" H 2050 1550 60  0000 C CNN
@@
 	2050 1550 2050 1400
 $Comp
-L C 47µ
+L C 47µ1
 U 1 1 5627D475
 P 1550 1250
-F 0 "47µ" H 1575 1350 50  0000 L CNN
+F 0 "47µ1" H 1575 1350 50  0000 L CNN
 F 1 "C" H 1575 1150 50  0000 L CNN
-F 2 "" H 1588 1100 30  0000 C CNN
+F 2 "Capacitors_ThroughHole:C_Axial_D6_L11_P18" H 1588 1100 30  0001 C CNN
 F 3 "" H 1550 1250 60  0000 C CNN
 	1    1550 1250
@@
 Connection ~ 2050 1400
 $Comp
-L C 33µ
+L C 33µ1
 U 1 1 5627D645
 P 2450 1250
-F 0 "33µ" H 2475 1350 50  0000 L CNN
+F 0 "33µ1" H 2475 1350 50  0000 L CNN
 F 1 "C" H 2475 1150 50  0000 L CNN
-F 2 "" H 2488 1100 30  0000 C CNN
+F 2 "Capacitors_ThroughHole:C_Radial_D5_L6_P2.5" H 2488 1100 30  0001 C CNN
 F 3 "" H 2450 1250 60  0000 C CNN
 	1    2450 1250
