File: KiCAD/Displayplatine/Display.sch (KiCad schematic (older format))
At the start: 14 parts, among them P1 CONN_01X08

Commit message: Displayplatine fertig + EADOG Footprint korrigiert
Parts:
- C1, C2, C3, C4, C5, C6, C7, C8, C9: footprint Capacitors_ThroughHole:C_Disc_D3_P2.5 -> Capacitors_ThroughHole:C_Disc_D7.5_P5
Changed lines of the file:
@@
 F 0 "C9" H 5725 4450 50  0000 L CNN
 F 1 "C" H 5725 4250 50  0000 L CNN
-F 2 "Capacitors_ThroughHole:C_Disc_D3_P2.5" H 5738 4200 30  0001 C CNN
+F 2 "Capacitors_ThroughHole:C_Disc_D7.5_P5" H 5738 4200 30  0001 C CNN
 F 3 "" H 5700 4350 60  0000 C CNN
 	1    5700 4350
@@
 F 0 "C8" H 5725 4250 50  0000 L CNN
 F 1 "C" H 5725 4050 50  0000 L CNN
-F 2 "Capacitors_ThroughHole:C_Disc_D3_P2.5" H 5738 4000 30  0001 C CNN
+F 2 "Capacitors_ThroughHole:C_Disc_D7.5_P5" H 5738 4000 30  0001 C CNN
 F 3 "" H 5700 4150 60  0000 C CNN
 	1    5700 4150
@@
 F 0 "C7" H 5725 4050 50  0000 L CNN
 F 1 "C" H 5725 3850 50  0000 L CNN
-F 2 "Capacitors_ThroughHole:C_Disc_D3_P2.5" H 5738 3800 30  0001 C CNN
+F 2 "Capacitors_ThroughHole:C_Disc_D7.5_P5" H 5738 3800 30  0001 C CNN
 F 3 "" H 5700 3950 60  0000 C CNN
 	1    5700 3950
@@
 F 0 "C6" H 5725 3850 50  0000 L CNN
 F 1 "C" H 5725 3650 50  0000 L CNN
-F 2 "Capacitors_ThroughHole:C_Disc_D3_P2.5" H 5738 3600 30  0001 C CNN
+F 2 "Capacitors_ThroughHole:C_Disc_D7.5_P5" H 5738 3600 30  0001 C CNN
 F 3 "" H 5700 3750 60  0000 C CNN
 	1    5700 3750
@@
 F 0 "C5" H 5725 3650 50  0000 L CNN
 F 1 "C" H 5725 3450 50  0000 L CNN
-F 2 "Capacitors_ThroughHole:C_Disc_D3_P2.5" H 5738 3400 30  0001 C CNN
+F 2 "Capacitors_ThroughHole:C_Disc_D7.5_P5" H 5738 3400 30  0001 C CNN
 F 3 "" H 5700 3550 60  0000 C CNN
 	1    5700 3550
@@
 F 0 "C4" H 5725 3450 50  0000 L CNN
 F 1 "C" H 5725 3250 50  0000 L CNN
-F 2 "Capacitors_ThroughHole:C_Disc_D3_P2.5" H 5738 3200 30  0001 C CNN
+F 2 "Capacitors_ThroughHole:C_Disc_D7.5_P5" H 5738 3200 30  0001 C CNN
 F 3 "" H 5700 3350 60  0000 C CNN
 	1    5700 3350
@@
 F 0 "C3" H 5725 3250 50  0000 L CNN
 F 1 "C" H 5725 3050 50  0000 L CNN
-F 2 "Capacitors_ThroughHole:C_Disc_D3_P2.5" H 5738 3000 30  0001 C CNN
+F 2 "Capacitors_ThroughHole:C_Disc_D7.5_P5" H 5738 3000 30  0001 C CNN
 F 3 "" H 5700 3150 60  0000 C CNN
 	1    5700 3150
@@
 F 0 "C2" H 5725 3050 50  0000 L CNN
 F 1 "C" H 5725 2850 50  0000 L CNN
-F 2 "Capacitors_ThroughHole:C_Disc_D3_P2.5" H 5738 2800 30  0001 C CNN
+F 2 "Capacitors_ThroughHole:C_Disc_D7.5_P5" H 5738 2800 30  0001 C CNN
 F 3 "" H 5700 2950 60  0000 C CNN
 	1    5700 2950
@@
 F 0 "C1" H 5725 2850 50  0000 L CNN
 F 1 "C" H 5725 2650 50  0000 L CNN
-F 2 "Capacitors_ThroughHole:C_Disc_D3_P2.5" H 5738 2600 30  0001 C CNN
+F 2 "Capacitors_ThroughHole:C_Disc_D7.5_P5" H 5738 2600 30  0001 C CNN
 F 3 "" H 5700 2750 60  0000 C CNN
 	1    5700 2750

Commit message: Displayplatine fertig
Parts:
- added P2, P3, P4, P5: CONN_01X01, Pin_Headers:Pin_Header_Straight_1x01, symbol CONN_01X01
Changed lines of the file:
@@
 Connection ~ 5850 3150
 Connection ~ 5850 2750
+$Comp
+L CONN_01X01 P2
+U 1 1 5630FB15
+P 7850 4450
+F 0 "P2" H 7850 4550 50  0000 C CNN
+F 1 "CONN_01X01" V 7950 4450 50  0000 C CNN
+F 2 "Pin_Headers:Pin_Header_Straight_1x01" H 7850 4450 60  0001 C CNN
+F 3 "" H 7850 4450 60  0000 C CNN
+	1    7850 4450
+	1    0    0    -1
+$EndComp
+$Comp
+L CONN_01X01 P3
+U 1 1 5630FB6B
+P 7850 4650
+F 0 "P3" H 7850 4750 50  0000 C CNN
+F 1 "CONN_01X01" V 7950 4650 50  0000 C CNN
+F 2 "Pin_Headers:Pin_Header_Straight_1x01" H 7850 4650 60  0001 C CNN
+F 3 "" H 7850 4650 60  0000 C CNN
+	1    7850 4650
+	1    0    0    -1
+$EndComp
+$Comp
+L CONN_01X01 P4
+U 1 1 5630FBB9
+P 7850 4850
+F 0 "P4" H 7850 4950 50  0000 C CNN
+F 1 "CONN_01X01" V 7950 4850 50  0000 C CNN
+F 2 "Pin_Headers:Pin_Header_Straight_1x01" H 7850 4850 60  0001 C CNN
+F 3 "" H 7850 4850 60  0000 C CNN
+	1    7850 4850
+	1    0    0    -1
+$EndComp
+$Comp
+L CONN_01X01 P5
+U 1 1 5630FC10
+P 7850 5050
+F 0 "P5" H 7850 5150 50  0000 C CNN
+F 1 "CONN_01X01" V 7950 5050 50  0000 C CNN
+F 2 "Pin_Headers:Pin_Header_Straight_1x01" H 7850 5050 60  0001 C CNN
+F 3 "" H 7850 5050 60  0000 C CNN
+	1    7850 5050
+	1    0    0    -1
+$EndComp
 $EndSCHEMATC

Commit message: Hauptplatine inkl TDA7266
Connections:
- net D1 renamed DISP-SI
- net D2 renamed DISP-SCL
- net D3 renamed DISP-A0
- net D4 renamed DISP-RST
- net D5 renamed DISP-CS1B
Changed lines of the file:
@@
 $EndComp
 Text GLabel 5650 2550 2    60   Input ~ 0
-D1
+DISP-SI
 Text GLabel 5650 2400 2    60   Input ~ 0
-D2
+DISP-SCL
 Text GLabel 5650 2250 2    60   Input ~ 0
-D3
+DISP-A0
 Text GLabel 5650 2100 2    60   Input ~ 0
-D4
+DISP-RST
 Text GLabel 5650 1950 2    60   Input ~ 0
-D5
+DISP-CS1B
 Text GLabel 6050 2650 2    60   Input ~ 0
 VCC
@@
 $EndComp
 Text GLabel 8200 2500 0    60   Input ~ 0
-D1
+DISP-SI
 Text GLabel 8200 2650 0    60   Input ~ 0
-D2
+DISP-SCL
 Text GLabel 8200 2800 0    60   Input ~ 0
-D3
+DISP-A0
 Text GLabel 8200 2950 0    60   Input ~ 0
-D4
+DISP-RST
 Text GLabel 8200 3100 0    60   Input ~ 0
-D5
+DISP-CS1B
 Text GLabel 8250 3250 0    60   Input ~ 0
 LED
